Commit message: add start pose and group state in rviz

File: src/dual_arm_moveit_config/config/dual_arm_real_v2.urdf.xacro (robot description, xacro)
@@ -39,4 +39,5 @@
     robot_ip="192.168.1.10"
     use_fake_hardware="$(arg use_fake_hardware)"
+    initial_positions="${dict(shoulder_pan_joint=-0.9579,shoulder_lift_joint=-1.9195,elbow_joint=2.5167,wrist_1_joint=-3.4194,wrist_2_joint=-2.0268,wrist_3_joint=0.2502)}"
     headless_mode="true"
     reverse_port="50002"
@@ -70,4 +71,5 @@
     robot_ip="192.168.1.20"
     use_fake_hardware="$(arg use_fake_hardware)"
+    initial_positions="${dict(shoulder_pan_joint=-2.155,shoulder_lift_joint=-1.4352,elbow_joint=-2.4564,wrist_1_joint=0.5894,wrist_2_joint=-4.1043,wrist_3_joint=-0.2312)}"
     headless_mode="true"
     reverse_port="50005"
@@ -95,4 +97,11 @@
       </material>
     </visual>
+    <collision>
+      <origin xyz="0 0 0" rpy="0 0 0"/>
+      <geometry>
+        <mesh filename="package://dual_arm_pkg/meshes/visual/cobot_frame_simple.stl"
+              scale="0.001 0.001 0.001"/>
+      </geometry>
+    </collision>
   </link>
 <joint name="table_to_cobot_frame" type="fixed">

Commit message: Add the consideration of gripper into URDF and generate the frame right_tcp

File: src/dual_arm_moveit_config/config/dual_arm_real_v2.urdf.xacro (robot description, xacro)
@@ -60,4 +60,11 @@
     <origin xyz="0 0 0.244" rpy="0 0 0"/>
   </joint>
+  <!-- Right TCP: fingertip gripping point 155 mm along +Z from right_tool0 -->
+  <link name="right_tcp"/>
+  <joint name="right_tool0_to_right_tcp" type="fixed">
+    <parent link="right_tool0"/>
+    <child  link="right_tcp"/>
+    <origin xyz="0 0 0.155" rpy="0 0 0"/>
+  </joint>
   <!-- ===================== RIGHT ARM ===================== -->
   <xacro:ur_robot

File: src/dual_arm_pkg/urdf/dual_arm.urdf.xacro (robot description, xacro)
@@ -476,4 +476,11 @@
     <child  link="left_tcp"/>
     <origin xyz="0 0 0.244" rpy="0 0 0"/>
+  </joint>
+  <!-- Right TCP: fingertip gripping point 155 mm along +Z from right_tool0 -->
+  <link name="right_tcp"/>
+  <joint name="right_tool0_to_right_tcp" type="fixed">
+    <parent link="right_tool0"/>
+    <child  link="right_tcp"/>
+    <origin xyz="0 0 0.155" rpy="0 0 0"/>
   </joint>
   <!-- RIGHT arm — right end of table -->

Commit message: Update the test scripts, the offset of the gripper

File: src/dual_arm_moveit_config/config/dual_arm_real_v2.urdf.xacro (robot description, xacro)
@@ -60,10 +60,10 @@
     <origin xyz="0 0 0.244" rpy="0 0 0"/>
   </joint>
-  <!-- Right TCP: fingertip gripping point 155 mm along +Z from right_tool0 -->
+  <!-- Right TCP: fingertip gripping point 150 mm along +Z from right_tool0 -->
   <link name="right_tcp"/>
   <joint name="right_tool0_to_right_tcp" type="fixed">
     <parent link="right_tool0"/>
     <child  link="right_tcp"/>
-    <origin xyz="0 0 0.155" rpy="0 0 0"/>
+    <origin xyz="-0.020 0 0.150" rpy="0 0 0"/>
   </joint>
   <!-- ===================== RIGHT ARM ===================== -->
